Commit message: 完善飞机结构，增加差动小车模型，增加摄像头

File: urdf/wheeled_robot.xacro (robot description, xacro)
@@ -1,4 +1,5 @@
 <?xml version="1.0" ?>
-<robot name="$(arg robot_name)" xmlns:xacro="http://www.ros.org/wiki/xacro">
+<robot name="$(arg robot_name)"
+  xmlns:xacro="http://www.ros.org/wiki/xacro">
   <xacro:property name="PI" value="3.1415926835897931"/>
   <xacro:property name="material_density" value="10.0"/>
@@ -14,6 +15,6 @@
   <!-- rear tyre -->
   <xacro:property name="rear_tyre_x" value="0.5"/>
-  <xacro:property name="rear_tyre_y" value="0.3"/>
-  <xacro:property name="rear_tyre_r" value="0.2"/>
+  <xacro:property name="rear_tyre_y" value="${base_width/2.0}"/>
+  <xacro:property name="rear_tyre_r" value="${base_collision_height/2.0}"/>
   <xacro:property name="rear_tyre_length" value="0.1"/>
   <xacro:property name="rear_tyre_mass" value="20"/>
@@ -23,7 +24,7 @@
   <!-- front tyre -->
   <xacro:property name="front_tyre_x" value="0.5"/>
-  <xacro:property name="front_tyre_y" value="0.3"/>
-  <xacro:property name="front_tyre_r" value="0.2"/>
-  <xacro:property name="front_tyre_length" value="0.1 "/>
+  <xacro:property name="front_tyre_y" value="${base_width/2.0}"/>
+  <xacro:property name="front_tyre_r" value="${base_collision_height/2.0}"/>
+  <xacro:property name="front_tyre_length" value="0.1"/>
   <xacro:property name="front_tyre_mass" value="20"/>
   <xacro:property name="front_tyre_mass_ixx" value="0.5"/>
@@ -40,31 +41,24 @@
   <!--Car Body-->
   <link name="base_link">
-    <collision>
+    <inertial>
       <origin xyz="0 0 ${base_collision_height}" rpy="0 0 0"/>
+      <mass value="${base_mass}"/>
+      <inertia ixx="${base_mass_ixx}" ixy="0" ixz="0" iyy="${base_mass_iyy}" iyz="0" izz="${base_mass_izz}" />
+    </inertial>
+    <visual>
+      <origin xyz="0 0 ${base_collision_height}" rpy="0 0 0" />
+      <geometry>
+        <box size="${base_length} ${base_width} ${base_height}" />
+      </geometry>
+      <material name="Yellow">
+        <color rgba="1.0 1.0 0.0 1.0"/>
+      </material>
+    </visual>
+    <collision>
+      <origin xyz="0 0 ${base_collision_height}" rpy="0 0 0"/>
       <geometry>
         <box size="${base_length} ${base_width} ${base_height}"/>
       </geometry>
     </collision>
-    <visual>
-      <origin xyz="0 0 ${base_collision_height}" rpy="0 0 0"/>
-      <geometry>
-        <box size="${base_length} ${base_width} ${base_height}"/>
-      </geometry>
-    </visual>
-  </link>
-  <joint name="inertial_joint" type="fixed">
-    <parent link="base_link"/>
-    <child link="main_mass"/>
-    <origin xyz="0 0 0" rpy="0 0 0"/>
-  </joint>
-  <link name="main_mass" type="fixed">
-    <inertial>
-      <origin xyz="0 0 0" rpy="0 0 0"/>
-      <mass value="${base_mass}"/>
-      <inertia
-        ixx="${base_mass_ixx}"  ixy="0.000000"  ixz="0.000000"
-        iyy="${base_mass_iyy}"  iyz="0.000000"
-        izz="${base_mass_izz}"/>
-    </inertial>
   </link>
   <!--velodyne VLP-16-->
@@ -116,4 +110,187 @@
     </sensor>
   </gazebo>
+  <!--Camera1 sensor-->
+  <joint name="camera1_joint" type="fixed">
+    <axis xyz="0 1 0" />
+    <origin xyz="${base_length/2-0.01} 0 ${base_height/2+base_collision_height+0.01}" rpy="0 0 0"/>
+    <parent link="base_link"/>
+    <child link="camera1_link"/>
+  </joint>
+  <link name="camera1_link">
+    <collision>
+      <origin xyz="0 0 0" rpy="0 0 0"/>
+      <geometry>
+        <box size="0.02 0.02 0.02"/>
+      </geometry>
+    </collision>
+    <visual>
+      <origin xyz="0 0 0" rpy="0 0 0"/>
+      <geometry>
+        <box size="0.02 0.02 0.02"/>
+      </geometry>
+      <material name="red" color="1 0 0 1"/>
+    </visual>
+  </link>
+  <gazebo reference="camera1_link">
+    <sensor type="camera" name="camera1">
+      <update_rate>30.0</update_rate>
+      <camera name="head">
+        <horizontal_fov>1.74532925</horizontal_fov>
+        <image>
+          <width>800</width>
+          <height>800</height>
+          <format>R8G8B8</format>
+        </image>
+        <clip>
+          <near>0.02</near>
+          <far>300</far>
+        </clip>
+        <noise>
+          <type>gaussian</type>
+          <!-- Noise is sampled independently per pixel on each frame.
+               That pixel's noise value is added to each of its color
+               channels, which at that point lie in the range [0,1]. -->
+          <mean>0.0</mean>
+          <stddev>0.007</stddev>
+        </noise>
+      </camera>
+      <plugin name="camera_controller" filename="libgazebo_ros_camera.so">
+        <alwaysOn>true</alwaysOn>
+        <updateRate>0.0</updateRate>
+        <cameraName>$(arg robot_name)/camera1</cameraName>
+        <imageTopicName>image_raw</imageTopicName>
+        <cameraInfoTopicName>camera_info</cameraInfoTopicName>
+        <frameName>camera_link</frameName>
+        <hackBaseline>0.07</hackBaseline>
+        <distortionK1>0.0</distortionK1>
+        <distortionK2>0.0</distortionK2>
+        <distortionK3>0.0</distortionK3>
+        <distortionT1>0.0</distortionT1>
+        <distortionT2>0.0</distortionT2>
+      </plugin>
+    </sensor>
+  </gazebo>
+  <!--Camera2 sensor-->
+  <joint name="camera2_joint" type="fixed">
+    <axis xyz="0 1 0" />
+    <origin xyz="0 ${base_width/2-0.01} ${base_height/2+base_collision_height+0.01}" rpy="0 0 1.570796"/>
+    <parent link="base_link"/>
+    <child link="camera2_link"/>
+  </joint>
+  <link name="camera2_link">
+    <collision>
+      <origin xyz="0 0 0" rpy="0 0 0"/>
+      <geometry>
+        <box size="0.02 0.02 0.02"/>
+      </geometry>
+    </collision>
+    <visual>
+      <origin xyz="0 0 0" rpy="0 0 0"/>
+      <geometry>
+        <box size="0.02 0.02 0.02"/>
+      </geometry>
+      <material name="red" color="1 0 0 1"/>
+    </visual>
+  </link>
+  <gazebo reference="camera2_link">
+    <sensor type="camera" name="camera2">
+      <update_rate>30.0</update_rate>
+      <camera name="head">
+        <horizontal_fov>1.74532925</horizontal_fov>
+        <image>
+          <width>800</width>
+          <height>800</height>
+          <format>R8G8B8</format>
+        </image>
+        <clip>
+          <near>0.02</near>
+          <far>300</far>
+        </clip>
+        <noise>
+          <type>gaussian</type>
+          <!-- Noise is sampled independently per pixel on each frame.
+               That pixel's noise value is added to each of its color
+               channels, which at that point lie in the range [0,1]. -->
+          <mean>0.0</mean>
+          <stddev>0.007</stddev>
+        </noise>
+      </camera>
+      <plugin name="camera_controller" filename="libgazebo_ros_camera.so">
+        <alwaysOn>true</alwaysOn>
+        <updateRate>0.0</updateRate>
+        <cameraName>$(arg robot_name)/camera2</cameraName>
+        <imageTopicName>image_raw</imageTopicName>
+        <cameraInfoTopicName>camera_info</cameraInfoTopicName>
+        <frameName>camera_link</frameName>
+        <hackBaseline>0.07</hackBaseline>
+        <distortionK1>0.0</distortionK1>
+        <distortionK2>0.0</distortionK2>
+        <distortionK3>0.0</distortionK3>
+        <distortionT1>0.0</distortionT1>
+        <distortionT2>0.0</distortionT2>
+      </plugin>
+    </sensor>
+  </gazebo>
+  <!--Camera3 sensor-->
+  <joint name="camera3_joint" type="fixed">
+    <axis xyz="0 1 0" />
+    <origin xyz="0 -${base_width/2-0.01} ${base_height/2+base_collision_height+0.01}" rpy="0 0 -1.570796"/>
+    <parent link="base_link"/>
+    <child link="camera3_link"/>
+  </joint>
+  <link name="camera3_link">
+    <collision>
+      <origin xyz="0 0 0" rpy="0 0 0"/>
+      <geometry>
+        <box size="0.02 0.02 0.02"/>
+      </geometry>
+    </collision>
+    <visual>
+      <origin xyz="0 0 0" rpy="0 0 0"/>
+      <geometry>
+        <box size="0.02 0.02 0.02"/>
+      </geometry>
+      <material name="red" color="1 0 0 1"/>
+    </visual>
+  </link>
+  <gazebo reference="camera3_link">
+    <sensor type="camera" name="camera3">
+      <update_rate>30.0</update_rate>
+      <camera name="head">
+        <horizontal_fov>1.74532925</horizontal_fov>
+        <image>
+          <width>800</width>
+          <height>800</height>
+          <format>R8G8B8</format>
+        </image>
+        <clip>
+          <near>0.02</near>
+          <far>300</far>
+        </clip>
+        <noise>
+          <type>gaussian</type>
+          <!-- Noise is sampled independently per pixel on each frame.
+               That pixel's noise value is added to each of its color
+               channels, which at that point lie in the range [0,1]. -->
+          <mean>0.0</mean>
+          <stddev>0.007</stddev>
+        </noise>
+      </camera>
+      <plugin name="camera_controller" filename="libgazebo_ros_camera.so">
+        <alwaysOn>true</alwaysOn>
+        <updateRate>0.0</updateRate>
+        <cameraName>$(arg robot_name)/camera3</cameraName>
+        <imageTopicName>image_raw</imageTopicName>
+        <cameraInfoTopicName>camera_info</cameraInfoTopicName>
+        <frameName>camera_link</frameName>
+        <hackBaseline>0.07</hackBaseline>
+        <distortionK1>0.0</distortionK1>
+        <distortionK2>0.0</distortionK2>
+        <distortionK3>0.0</distortionK3>
+        <distortionT1>0.0</distortionT1>
+        <distortionT2>0.0</distortionT2>
+      </plugin>
+    </sensor>
+  </gazebo>
   <!--Rear Right Wheel-->
   <joint name="rear_right_wheel_joint" type="continuous">
@@ -142,8 +319,5 @@
       <origin xyz="0 0 0" rpy="0 0 0"/>
       <mass value="${rear_tyre_mass}"/>
-      <inertia
-        ixx="${rear_tyre_mass_ixx}"  ixy="0.000000"  ixz="0.000000"
-        iyy="${rear_tyre_mass_iyy}"  iyz="0.000000"
-        izz="${rear_tyre_mass_izz}"/>
+      <inertia ixx="${rear_tyre_mass_ixx}" ixy="0.000000" ixz="0.000000" iyy="${rear_tyre_mass_iyy}" iyz="0.000000" izz="${rear_tyre_mass_izz}"/>
     </inertial>
   </link>
@@ -174,8 +348,5 @@
       <origin xyz="0 0 0" rpy="0 0 0"/>
       <mass value="${rear_tyre_mass}"/>
-      <inertia
-        ixx="${rear_tyre_mass_ixx}"  ixy="0.000000"  ixz="0.000000"
-        iyy="${rear_tyre_mass_iyy}"  iyz="0.000000"
-        izz="${rear_tyre_mass_izz}"/>
+      <inertia ixx="${rear_tyre_mass_ixx}" ixy="0.000000" ixz="0.000000" iyy="${rear_tyre_mass_iyy}" iyz="0.000000" izz="${rear_tyre_mass_izz}"/>
     </inertial>
   </link>
@@ -199,11 +370,7 @@
       <origin xyz="0 0 0" rpy="0 0 0"/>
       <mass value="${str_mass}"/>
-      <inertia
-      ixx="${str_mass_ixx}"  ixy="0.000000"  ixz="0.000000"
-      iyy="${str_mass_iyy}"  iyz="0.000000"
-      izz="${str_mass_izz}"/>
-    </inertial>
-  </link>
-  <!--Front Right Wheel-->
+      <inertia ixx="${str_mass_ixx}" ixy="0.000000" ixz="0.000000" iyy="${str_mass_iyy}" iyz="0.000000" izz="${str_mass_izz}"/>
+    </inertial>
+  </link>  <!--Front Right Wheel-->
   <joint name="front_right_wheel_joint" type="continuous">
     <parent link="front_right_steering_link"/>
@@ -231,8 +398,5 @@
       <origin xyz="0 0 0" rpy="0 0 0"/>
       <mass value="${front_tyre_mass}"/>
-      <inertia
-        ixx="${front_tyre_mass_ixx}"  ixy="0.000000"  ixz="0.000000"
-        iyy="${front_tyre_mass_iyy}"  iyz="0.000000"
-        izz="${front_tyre_mass_izz}"/>
+      <inertia ixx="${front_tyre_mass_ixx}" ixy="0.000000" ixz="0.000000" iyy="${front_tyre_mass_iyy}" iyz="0.000000" izz="${front_tyre_mass_izz}"/>
     </inertial>
   </link>
@@ -256,11 +420,7 @@
       <origin xyz="0 0 0" rpy="0 0 0"/>
       <mass value="${str_mass}"/>
-      <inertia
-      ixx="${str_mass_ixx}"  ixy="0.000000"  ixz="0.000000"
-      iyy="${str_mass_iyy}"  iyz="0.000000"
-      izz="${str_mass_izz}"/>
-    </inertial>
-  </link>
-  <!--Front Left Wheel-->
+      <inertia ixx="${str_mass_ixx}" ixy="0.000000" ixz="0.000000" iyy="${str_mass_iyy}" iyz="0.000000" izz="${str_mass_izz}"/>
+    </inertial>
+  </link>  <!--Front Left Wheel-->
   <joint name="front_left_wheel_joint" type="continuous">
     <parent link="front_left_steering_link"/>
@@ -288,11 +448,7 @@
       <origin xyz="0 0 0" rpy="0 0 0"/>
       <mass value="${front_tyre_mass}"/>
-      <inertia
-        ixx="${front_tyre_mass_ixx}"  ixy="0.000000"  ixz="0.000000"
-        iyy="${front_tyre_mass_iyy}"  iyz="0.000000"
-        izz="${front_tyre_mass_izz}"/>
-    </inertial>
-  </link>
-  <!-- motors and transmissions for the two rear wheels -->
+      <inertia ixx="${front_tyre_mass_ixx}" ixy="0.000000" ixz="0.000000" iyy="${front_tyre_mass_iyy}" iyz="0.000000" izz="${front_tyre_mass_izz}"/>
+    </inertial>
+  </link>  <!-- motors and transmissions for the two rear wheels -->
   <transmission name="tran1">
     <type>transmission_interface/SimpleTransmission</type>
@@ -314,6 +470,5 @@
       <mechanicalReduction>1</mechanicalReduction>
     </actuator>
-  </transmission>
-  <!-- EPS and transmissions for the front steering -->
+  </transmission>  <!-- EPS and transmissions for the front steering -->
   <transmission name="tran3">
     <type>transmission_interface/SimpleTransmission</type>
@@ -337,6 +492,5 @@
       <motorTorqueConstant>1000000</motorTorqueConstant>
     </actuator>
-  </transmission>
-  <!-- Friction Parametres -->
+  </transmission>  <!-- Friction Parametres -->
   <gazebo reference="rear_right_wheel_link">
     <mu1>10000000</mu1>
@@ -362,6 +516,5 @@
     <kp>10000000</kp>
     <kd>1</kd>
-  </gazebo>
-  <!-- Gazebo Plugins -->
+  </gazebo>  <!-- Gazebo Plugins -->
   <gazebo>
     <plugin name="gazebo_ros_control" filename="libgazebo_ros_control.so">
