Commit message: 添加IMU滤波和预积分的python代码

File: urdf/tracked_robot.xacro (robot description, xacro)
@@ -1,5 +1,6 @@
 <?xml version="1.0" ?>
-<robot name="$(arg robot_name)"
+<robot name="airport_robot"
     xmlns:xacro="http://www.ros.org/wiki/xacro">
+    <xacro:property name="robot_name" value="airport_robot"/>
     <xacro:property name="PI" value="3.1415926835897931"/>
     <xacro:property name="material_density" value="10.0"/>
@@ -39,4 +40,12 @@
     <xacro:property name="str_mass_iyy" value="0.025"/>
     <xacro:property name="str_mass_izz" value="0.012"/>
+    <!-- To fix the problem -->
+    <!-- The root link base_link has an inertia specified in the URDF, but KDL does not support a root link with an inertia.  As a workaround, you can add an extra dummy link to your URDF. -->
+    <link name="dummy">
+    </link>
+    <joint name="dummy_joint" type="fixed">
+        <parent link="dummy"/>
+        <child link="base_link"/>
+    </joint>
     <!--Car Body-->
     <link name="base_link">
@@ -68,5 +77,6 @@
     <xacro:property name="organize_cloud" value="$(arg organize_cloud)" />
     <xacro:include filename="$(find velodyne_description)/urdf/VLP-16.urdf.xacro"/>
-    <xacro:VLP-16 parent="base_link" name="velodyne" topic="/velodyne_points" organize_cloud="${organize_cloud}" hz="10" samples="440" gpu="${gpu}">
+    <xacro:VLP-16 parent="base_link" name="velodyne" topic="/points_raw" organize_cloud="${organize_cloud}" hz="11" samples="440" gpu="${gpu}">
+        <!-- <origin xyz="${base_length/2.0-0.08} 0 0.72" rpy="0 ${PI/12} 0" /> -->
         <origin xyz="0 0 0.8" rpy="0 0 0" />
     </xacro:VLP-16>
@@ -95,15 +105,14 @@
         <sensor name="imu_sensor" type="imu">
             <always_on>true</always_on>
-            <update_rate>100</update_rate>
+            <update_rate>200.0</update_rate>
             <visualize>true</visualize>
             <topic>__default_topic__</topic>
             <plugin filename="libgazebo_ros_imu_sensor.so" name="imu_plugin">
                 <topicName>/imu</topicName>
-                <bodyName>imu_link</bodyName>
-                <updateRateHZ>2.0</updateRateHZ>
-                <gaussianNoise>0.0</gaussianNoise>
+                <frameName>imu_link</frameName>
+                <updateRateHZ>200.0</updateRateHZ>
+                <gaussianNoise>0.001</gaussianNoise>
                 <xyzOffset>0 0 0</xyzOffset>
                 <rpyOffset>0 0 0</rpyOffset>
-                <frameName>imu_link</frameName>
             </plugin>
             <pose>0 0 0 0 0 0</pose>
@@ -158,5 +167,5 @@
                 <alwaysOn>true</alwaysOn>
                 <updateRate>0.0</updateRate>
-                <cameraName>$(arg robot_name)/camera1</cameraName>
+                <cameraName>${robot_name}/camera1</cameraName>
                 <imageTopicName>image_raw</imageTopicName>
                 <cameraInfoTopicName>camera_info</cameraInfoTopicName>
@@ -219,5 +228,5 @@
                 <alwaysOn>true</alwaysOn>
                 <updateRate>0.0</updateRate>
-                <cameraName>$(arg robot_name)/camera2</cameraName>
+                <cameraName>${robot_name}/camera2</cameraName>
                 <imageTopicName>image_raw</imageTopicName>
                 <cameraInfoTopicName>camera_info</cameraInfoTopicName>
@@ -280,5 +289,5 @@
                 <alwaysOn>true</alwaysOn>
                 <updateRate>0.0</updateRate>
-                <cameraName>$(arg robot_name)/camera3</cameraName>
+                <cameraName>${robot_name}/camera3</cameraName>
                 <imageTopicName>image_raw</imageTopicName>
                 <cameraInfoTopicName>camera_info</cameraInfoTopicName>
@@ -479,5 +488,5 @@
     <gazebo>
         <plugin name="gazebo_ros_control" filename="libgazebo_ros_control.so">
-            <robotNamespace>/$(arg robot_name)</robotNamespace>
+            <robotNamespace>/${robot_name}</robotNamespace>
             <robotParam>robot_description</robotParam>
             <robotSimType>gazebo_ros_control/DefaultRobotHWSim</robotSimType>
@@ -488,5 +497,5 @@
             <jointName>rear_left_wheel_joint, rear_right_wheel_joint, front_right_wheel_joint, front_left_wheel_joint</jointName>
             <updateRate>50.0</updateRate>
-            <robotNamespace>/$(arg robot_name)</robotNamespace>
+            <robotNamespace>/${robot_name}</robotNamespace>
             <alwaysOn>true</alwaysOn>
         </plugin>

File: urdf/wheeled_robot.xacro (robot description, xacro)
@@ -14,5 +14,5 @@
   <xacro:property name="base_mass_izz" value="${(base_width*base_width+base_width*base_width)*base_mass/12.0}"/>
   <!-- rear tyre -->
-  <xacro:property name="rear_tyre_x" value="0.5"/>
+  <xacro:property name="rear_tyre_x" value="${base_length/2.0}"/>
   <xacro:property name="rear_tyre_y" value="${base_width/2.0}"/>
   <xacro:property name="rear_tyre_r" value="${base_collision_height/2.0}"/>
@@ -23,5 +23,5 @@
   <xacro:property name="rear_tyre_mass_izz" value="0.5"/>
   <!-- front tyre -->
-  <xacro:property name="front_tyre_x" value="0.5"/>
+  <xacro:property name="front_tyre_x" value="${base_length/2.0}"/>
   <xacro:property name="front_tyre_y" value="${base_width/2.0}"/>
   <xacro:property name="front_tyre_r" value="${base_collision_height/2.0}"/>
@@ -69,5 +69,5 @@
   <xacro:include filename="$(find velodyne_description)/urdf/VLP-16.urdf.xacro"/>
   <xacro:VLP-16 parent="base_link" name="velodyne" topic="/velodyne_points" organize_cloud="${organize_cloud}" hz="10" samples="440" gpu="${gpu}">
-    <origin xyz="0 0 0.8" rpy="0 0 0" />
+    <origin xyz="${base_length/2.0} 0 0.64" rpy="0 ${PI/12} 0" />
   </xacro:VLP-16>
   <!--IMU sensor-->
@@ -95,5 +95,5 @@
     <sensor name="imu_sensor" type="imu">
       <always_on>true</always_on>
-      <update_rate>100</update_rate>
+      <update_rate>200</update_rate>
       <visualize>true</visualize>
       <topic>__default_topic__</topic>
