Commit message: 完成cartogpher配置

File: urdf/tracked_robot copy.xacro (robot description, xacro)
@@ -42,10 +42,9 @@
     <!-- To fix the problem -->
     <!-- The root link base_link has an inertia specified in the URDF, but KDL does not support a root link with an inertia.  As a workaround, you can add an extra dummy link to your URDF. -->
-    <link name="base_footprint">
-    </link>
-    <joint name="base_joint" type="fixed">
-        <parent link="base_footprint"/>
+    <link name="dummy">
+    </link>
+    <joint name="dummy_joint" type="fixed">
+        <parent link="dummy"/>
         <child link="base_link"/>
-        <origin xyz="0 0 0" rpy="0 0 0"/>
     </joint>
     <!--Car Body-->
@@ -82,5 +81,5 @@
         <origin xyz="0 0 0.8" rpy="0 0 0" />
     </xacro:VLP-16>
-    <!-- IMU sensor
+    <!--IMU sensor-->
     <joint name="imu_joint" type="fixed">
         <parent link="base_link"/>
@@ -119,85 +118,5 @@
             <pose>0 0 0 0 0 0</pose>
         </sensor>
-    </gazebo> -->
-    <gazebo>
-        <plugin name="p3d_base_controller" filename="libgazebo_ros_p3d.so">
-            <alwaysOn>true</alwaysOn>
-            <updateRate>10.0</updateRate>
-            <bodyName>base_link</bodyName>
-            <topicName>odom</topicName>
-            <gaussianNoise>0</gaussianNoise>
-            <frameName>world</frameName>
-            <xyzOffsets>0 0 0</xyzOffsets>
-            <rpyOffsets>0 0 0</rpyOffsets>
-        </plugin>
-    </gazebo>
-    <!--Laser sensor-->
-    <xacro:macro name="laser_block" params="index min_range *origin">
-        <joint name="laser${index}_joint" type="fixed">
-            <xacro:insert_block name="origin" />
-            <parent link="base_link"/>
-            <child link="laser${index}_link"/>
-        </joint>
-        <link name="laser${index}_link">
-            <collision>
-                <origin xyz="0 0 0" rpy="0 0 0"/>
-                <geometry>
-                    <cylinder length="0.05" radius="0.05"/>
-                </geometry>
-            </collision>
-            <visual>
-                <origin xyz="0 0 0" rpy="0 0 0"/>
-                <geometry>
-                    <cylinder length="0.05" radius="0.05"/>
-                </geometry>
-                <material name="Green">
-                    <color rgba="0 1.0 0.0 1.0"/>
-                </material>
-            </visual>
-        </link>
-        <gazebo reference="laser${index}_link">
-            <sensor type="ray" name="laser${index}_sensor">
-                <pose>0 0 0 0 0 0</pose>
-                <visualize>false</visualize>
-                <update_rate>10</update_rate>
-                <ray>
-                    <scan>
-                        <horizontal>
-                            <samples>920</samples>
-                            <resolution>0.391</resolution>
-                            <min_angle>-3.1415926</min_angle>
-                            <max_angle>3.1415926</max_angle>
-                        </horizontal>
-                    </scan>
-                    <range>
-                        <min>${min_range}</min>
-                        <max>40.0</max>
-                        <resolution>0.03</resolution>
-                    </range>
-                    <noise>
-                        <type>gaussian</type>
-                        <mean>0.0</mean>
-                        <stddev>0.05</stddev>
-                    </noise>
-                </ray>
-                <plugin name="gazebo_ros_laser${index}_controller" filename="libgazebo_ros_laser.so">
-                    <topicName>/scan_raw${index}</topicName>
-                    <frameName>laser${index}_link</frameName>
-                </plugin>
-            </sensor>
-        </gazebo>
-    </xacro:macro>
-    <xacro:laser_block index="_1" min_range="1.3">
-        <origin xyz="${base_length/2} ${base_width/2} 0.5" rpy="0 0 0"/>
-    </xacro:laser_block>
-    <xacro:laser_block index="_2" min_range="1.3">
-        <origin xyz="${base_length/2} ${-base_width/2} 0.5" rpy="0 0 0"/>
-    </xacro:laser_block>
-    <xacro:laser_block index="_3" min_range="1.3">
-        <origin xyz="${-base_length/2} ${base_width/2} 0.5" rpy="0 0 0"/>
-    </xacro:laser_block>
-    <xacro:laser_block index="_4" min_range="1.3">
-        <origin xyz="${-base_length/2} ${-base_width/2} 0.5" rpy="0 0 0"/>
-    </xacro:laser_block>
+    </gazebo>
     <!--Camera1 sensor-->
     <joint name="camera1_joint" type="fixed">

File: urdf/wheeled_robot.xacro (robot description, xacro)
@@ -39,4 +39,12 @@
   <xacro:property name="str_mass_iyy" value="0.025"/>
   <xacro:property name="str_mass_izz" value="0.012"/>
+  <!-- To fix the problem -->
+  <!-- The root link base_link has an inertia specified in the URDF, but KDL does not support a root link with an inertia.  As a workaround, you can add an extra dummy link to your URDF. -->
+  <link name="dummy">
+  </link>
+  <joint name="dummy_joint" type="fixed">
+    <parent link="dummy"/>
+    <child link="base_link"/>
+  </joint>
   <!--Car Body-->
   <link name="base_link">
@@ -68,11 +76,17 @@
   <xacro:property name="organize_cloud" value="$(arg organize_cloud)" />
   <xacro:include filename="$(find velodyne_description)/urdf/VLP-16.urdf.xacro"/>
-  <xacro:VLP-16 parent="base_link" name="velodyne" topic="/velodyne_points" organize_cloud="${organize_cloud}" hz="10" samples="440" gpu="${gpu}">
-    <origin xyz="${base_length/2.0} 0 0.64" rpy="0 ${PI/12} 0" />
+  <xacro:VLP-16 parent="base_link" name="velodyne" topic="/points_raw" organize_cloud="${organize_cloud}" hz="11" samples="440" gpu="${gpu}">
+    <!-- <origin xyz="${base_length/2.0-0.08} 0 0.72" rpy="0 ${PI/12} 0" /> -->
+    <origin xyz="0 0 0.8" rpy="0 0 0" />
   </xacro:VLP-16>
   <!--IMU sensor-->
+  <joint name="imu_joint" type="fixed">
+    <parent link="base_link"/>
+    <child link="imu_link"/>
+    <origin xyz="0 0 ${base_collision_height}" rpy="0 0 0"/>
+  </joint>
   <link name="imu_link">
     <collision>
-      <origin xyz="0 0 0.4" rpy="0 0 0"/>
+      <origin xyz="0 0 0" rpy="0 0 0"/>
       <geometry>
         <box size="0.1 0.1 0.1"/>
@@ -80,5 +94,5 @@
     </collision>
     <visual>
-      <origin xyz="0 0 0.4" rpy="0 0 0"/>
+      <origin xyz="0 0 0" rpy="0 0 0"/>
       <geometry>
         <box size="0.1 0.1 0.1"/>
@@ -86,24 +100,18 @@
     </visual>
   </link>
-  <joint name="imu_joint" type="fixed">
-    <parent link="base_link"/>
-    <child link="imu_link"/>
-    <origin xyz="0 0 0" rpy="0 0 0"/>
-  </joint>
   <gazebo reference="imu_link">
     <gravity>true</gravity>
     <sensor name="imu_sensor" type="imu">
       <always_on>true</always_on>
-      <update_rate>200</update_rate>
+      <update_rate>200.0</update_rate>
       <visualize>true</visualize>
       <topic>__default_topic__</topic>
       <plugin filename="libgazebo_ros_imu_sensor.so" name="imu_plugin">
         <topicName>/imu</topicName>
-        <bodyName>imu_link</bodyName>
-        <updateRateHZ>2.0</updateRateHZ>
+        <frameName>imu_link</frameName>
+        <updateRateHZ>200.0</updateRateHZ>
         <gaussianNoise>0.0</gaussianNoise>
         <xyzOffset>0 0 0</xyzOffset>
         <rpyOffset>0 0 0</rpyOffset>
-        <frameName>imu_link</frameName>
       </plugin>
       <pose>0 0 0 0 0 0</pose>
@@ -450,5 +458,6 @@
       <inertia ixx="${front_tyre_mass_ixx}" ixy="0.000000" ixz="0.000000" iyy="${front_tyre_mass_iyy}" iyz="0.000000" izz="${front_tyre_mass_izz}"/>
     </inertial>
-  </link>  <!-- motors and transmissions for the two rear wheels -->
+  </link>
+  <!-- motors and transmissions for the two rear wheels -->
   <transmission name="tran1">
     <type>transmission_interface/SimpleTransmission</type>
@@ -470,5 +479,6 @@
       <mechanicalReduction>1</mechanicalReduction>
     </actuator>
-  </transmission>  <!-- EPS and transmissions for the front steering -->
+  </transmission>
+  <!-- EPS and transmissions for the front steering -->
   <transmission name="tran3">
     <type>transmission_interface/SimpleTransmission</type>
@@ -492,5 +502,6 @@
       <motorTorqueConstant>1000000</motorTorqueConstant>
     </actuator>
-  </transmission>  <!-- Friction Parametres -->
+  </transmission>
+  <!-- Friction Parametres -->
   <gazebo reference="rear_right_wheel_link">
     <mu1>10000000</mu1>
@@ -516,5 +527,6 @@
     <kp>10000000</kp>
     <kd>1</kd>
-  </gazebo>  <!-- Gazebo Plugins -->
+  </gazebo>
+  <!-- Gazebo Plugins -->
   <gazebo>
     <plugin name="gazebo_ros_control" filename="libgazebo_ros_control.so">
